Commit message: [ Turtlebot Addition ] : Adds another turtlebot and all three are now independent from each other

File: turtlebots/urdf/turtlebot3_burger_3.gazebo.xacro (robot description, xacro)
@@ -1,10 +1,10 @@
 <?xml version="1.0"?>
-<robot name="turtlebot3_burger_sim_tb1" xmlns:xacro="http://ros.org/wiki/xacro">
+<robot name="turtlebot3_burger_sim_tb2" xmlns:xacro="http://ros.org/wiki/xacro">
   <xacro:arg name="laser_visual" default="false"/>
   <xacro:arg name="imu_visual"   default="false"/>
-  <gazebo reference="base_link_tb1">
+  <gazebo reference="base_link_tb2">
     <material>Gazebo/DarkGrey</material>
   </gazebo>
-  <gazebo reference="wheel_left_link_tb1">
+  <gazebo reference="wheel_left_link_tb2">
     <mu1>0.1</mu1>
     <mu2>0.1</mu2>
@@ -16,5 +16,5 @@
     <material>Gazebo/FlatBlack</material>
   </gazebo>
-  <gazebo reference="wheel_right_link_tb1">
+  <gazebo reference="wheel_right_link_tb2">
     <mu1>0.1</mu1>
     <mu2>0.1</mu2>
@@ -26,5 +26,5 @@
     <material>Gazebo/FlatBlack</material>
   </gazebo>
-  <gazebo reference="caster_back_link_tb1">
+  <gazebo reference="caster_back_link_tb2">
     <mu1>0.1</mu1>
     <mu2>0.1</mu2>
@@ -35,5 +35,5 @@
     <material>Gazebo/FlatBlack</material>
   </gazebo>
-  <gazebo reference="imu_link_tb1">
+  <gazebo reference="imu_link_tb2">
     <sensor type="imu" name="imu">
       <always_on>true</always_on>
@@ -44,7 +44,7 @@
   <gazebo>
     <plugin name="turtlebot3_burger_controller" filename="libgazebo_ros_diff_drive.so">
-      <commandTopic>cmd_vel_tb1</commandTopic>
-      <odometryTopic>odom_tb1</odometryTopic>
-      <odometryFrame>odom_tb1</odometryFrame>
+      <commandTopic>cmd_vel_tb2</commandTopic>
+      <odometryTopic>odom_tb2</odometryTopic>
+      <odometryFrame>odom_tb2</odometryFrame>
       <odometrySource>world</odometrySource>
       <publishOdomTF>true</publishOdomTF>
@@ -55,6 +55,6 @@
       <legacyMode>false</legacyMode>
       <updateRate>30</updateRate>
-      <leftJoint>wheel_left_joint_tb1</leftJoint>
-      <rightJoint>wheel_right_joint_tb1</rightJoint>
+      <leftJoint>wheel_left_joint_tb2</leftJoint>
+      <rightJoint>wheel_right_joint_tb2</rightJoint>
       <wheelSeparation>0.160</wheelSeparation>
       <wheelDiameter>0.066</wheelDiameter>
@@ -67,8 +67,8 @@
     <plugin name="imu_plugin" filename="libgazebo_ros_imu.so">
       <alwaysOn>true</alwaysOn>
-      <bodyName>imu_link_tb1</bodyName>
-      <frameName>imu_link_tb1</frameName>
-      <topicName>imu_tb1</topicName>
-      <serviceName>imu_service_tb1</serviceName>
+      <bodyName>imu_link_tb2</bodyName>
+      <frameName>imu_link_tb2</frameName>
+      <topicName>imu_tb2</topicName>
+      <serviceName>imu_service_tb2</serviceName>
       <gaussianNoise>0.0</gaussianNoise>
       <updateRate>0</updateRate>
@@ -92,5 +92,5 @@
     </plugin>
   </gazebo>
-  <gazebo reference="base_scan_tb1">
+  <gazebo reference="base_scan_tb2">
     <material>Gazebo/FlatBlack</material>
     <sensor type="ray" name="lds_lfcd_sensor">
@@ -119,6 +119,6 @@
       </ray>
       <plugin name="gazebo_ros_lds_lfcd_controller" filename="libgazebo_ros_laser.so">
-        <topicName>scan_tb1</topicName>
-        <frameName>base_scan_tb1</frameName>
+        <topicName>scan_tb2</topicName>
+        <frameName>base_scan_tb2</frameName>
       </plugin>
     </sensor>

File: turtlebots/urdf/turtlebot3_burger_3.urdf.xacro (robot description, xacro)
@@ -1,13 +1,13 @@
 <?xml version="1.0" ?>
-<robot name="turtlebot3_burger_tb1" xmlns:xacro="http://ros.org/wiki/xacro">
+<robot name="turtlebot3_burger_tb2" xmlns:xacro="http://ros.org/wiki/xacro">
   <xacro:include filename="$(find turtlebots)/urdf/common_properties.xacro"/>
-  <xacro:include filename="$(find turtlebots)/urdf/turtlebot3_burger.gazebo.xacro"/>
+  <xacro:include filename="$(find turtlebots)/urdf/turtlebot3_burger_3.gazebo.xacro"/>
   <link name="base_footprint"/>
   <joint name="base_joint" type="fixed">
     <parent link="base_footprint"/>
-    <child link="base_link_tb1"/>
+    <child link="base_link_tb2"/>
     <origin xyz="0.0 0.0 0.010" rpy="0 0 0"/>
   </joint>
-  <link name="base_link_tb1">
+  <link name="base_link_tb2">
     <visual>
       <origin xyz="-0.032 0 0.0" rpy="0 0 0"/>
@@ -31,11 +31,11 @@
     </inertial>
   </link>
-  <joint name="wheel_left_joint_tb1" type="continuous">
-    <parent link="base_link_tb1"/>
-    <child link="wheel_left_link_tb1"/>
+  <joint name="wheel_left_joint_tb2" type="continuous">
+    <parent link="base_link_tb2"/>
+    <child link="wheel_left_link_tb2"/>
     <origin xyz="0.0 0.08 0.023" rpy="-1.57 0 0"/>
     <axis xyz="0 0 1"/>
   </joint>
-  <link name="wheel_left_link_tb1">
+  <link name="wheel_left_link_tb2">
     <visual>
       <origin xyz="0 0 0" rpy="1.57 0 0"/>
@@ -59,11 +59,11 @@
       </inertial>
   </link>
-  <joint name="wheel_right_joint_tb1" type="continuous">
-    <parent link="base_link_tb1"/>
-    <child link="wheel_right_link_tb1"/>
+  <joint name="wheel_right_joint_tb2" type="continuous">
+    <parent link="base_link_tb2"/>
+    <child link="wheel_right_link_tb2"/>
     <origin xyz="0.0 -0.080 0.023" rpy="-1.57 0 0"/>
     <axis xyz="0 0 1"/>
   </joint>
-  <link name="wheel_right_link_tb1">
+  <link name="wheel_right_link_tb2">
     <visual>
       <origin xyz="0 0 0" rpy="1.57 0 0"/>
@@ -87,10 +87,10 @@
       </inertial>
   </link>
-  <joint name="caster_back_joint_tb1" type="fixed">
-    <parent link="base_link_tb1"/>
-    <child link="caster_back_link_tb1"/>
+  <joint name="caster_back_joint_tb2" type="fixed">
+    <parent link="base_link_tb2"/>
+    <child link="caster_back_link_tb2"/>
     <origin xyz="-0.081 0 -0.004" rpy="-1.57 0 0"/>
   </joint>
-  <link name="caster_back_link_tb1">
+  <link name="caster_back_link_tb2">
     <collision>
       <origin xyz="0 0.001 0" rpy="0 0 0"/>
@@ -107,16 +107,16 @@
     </inertial>
   </link>
-  <joint name="imu_joint_tb1" type="fixed">
-    <parent link="base_link_tb1"/>
-    <child link="imu_link_tb1"/>
+  <joint name="imu_joint_tb2" type="fixed">
+    <parent link="base_link_tb2"/>
+    <child link="imu_link_tb2"/>
     <origin xyz="-0.032 0 0.068" rpy="0 0 0"/>
   </joint>
-  <link name="imu_link_tb1"/>
-  <joint name="scan_joint_tb1" type="fixed">
-    <parent link="base_link_tb1"/>
-    <child link="base_scan_tb1"/>
+  <link name="imu_link_tb2"/>
+  <joint name="scan_joint_tb2" type="fixed">
+    <parent link="base_link_tb2"/>
+    <child link="base_scan_tb2"/>
     <origin xyz="-0.032 0 0.172" rpy="0 0 0"/>
   </joint>
-  <link name="base_scan_tb1">
+  <link name="base_scan_tb2">
     <visual>
       <origin xyz="0 0 0.0" rpy="0 0 0"/>
